Commit message: feat: Add assets for demo test

File: cobot3_ws/isaacpjt/smart_farm/assets/simple_pallet.urdf (robot description, URDF)
Before this commit: robot pallet_simplified, 1 links, 0 joints
Links:
- link pallet_link: geometry collision box size=0.40 0.04 0.07; collision box size=0.40 0.04 0.07
